Commit message: Create tesseract_environment and semi-isolate

File: tesseract_environment/test/urdf/lbr_iiwa_14_r820.urdf (robot description, URDF)
Before this commit: robot kuka_lbr_iiwa_14_r820, 10 links, 9 joints
Links:
- link base_link: geometry collision mesh filename=package://tesseract_environment/test/urdf/lbr_iiwa_14_r820/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; visual mesh filename=package://tesseract_environment/test/urdf/lbr_iiwa_14_r820/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
- link link_1: geometry collision mesh filename=package://tesseract_environment/test/urdf/lbr_iiwa_14_r820/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; visual mesh filename=package://tesseract_environment/test/urdf/lbr_iiwa_14_r820/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
- link link_2: geometry collision mesh filename=package://tesseract_environment/test/urdf/lbr_iiwa_14_r820/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; visual mesh filename=package://tesseract_environment/test/urdf/lbr_iiwa_14_r820/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
- link link_3: geometry collision mesh filename=package://tesseract_environment/test/urdf/lbr_iiwa_14_r820/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; visual mesh filename=package://tesseract_environment/test/urdf/lbr_iiwa_14_r820/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
- link link_4: geometry collision mesh filename=package://tesseract_environment/test/urdf/lbr_iiwa_14_r820/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; visual mesh filename=package://tesseract_environment/test/urdf/lbr_iiwa_14_r820/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
- link link_5: geometry collision mesh filename=package://tesseract_environment/test/urdf/lbr_iiwa_14_r820/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; visual mesh filename=package://tesseract_environment/test/urdf/lbr_iiwa_14_r820/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
- link link_6: geometry collision mesh filename=package://tesseract_environment/test/urdf/lbr_iiwa_14_r820/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; visual mesh filename=package://tesseract_environment/test/urdf/lbr_iiwa_14_r820/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
- link link_7: geometry collision mesh filename=package://tesseract_environment/test/urdf/lbr_iiwa_14_r820/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; visual mesh filename=package://tesseract_environment/test/urdf/lbr_iiwa_14_r820/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
